File: PCB/Css.kicad_pcb (KiCad board)
At the start: 2 copper layers, 84.5 x 92 mm, 12 parts, among them U1 ESP32-S3-MINI-1, U2 LM358

Commit message: Some PCB changes
Parts:
- moved C1 20.3 mm to (108.5, 87.0), turned to -90 degrees
- moved C2 19.1 mm to (127.5, 28.5), turned to 180 degrees
- moved R6 15.6 mm to (162.5, 52.9)
- moved R3 15.3 mm to (149.8, 88.0)
- moved R5 11.2 mm to (122.8, 54.0)
Routing:
- net +5VA: track 130.0 -> 83.5 mm, vias 1 -> 0
- net Net-(MK1-+): track 91.7 -> 71.1 mm
- net Net-(C1-Pad2): track 8.15 -> 26.4 mm
- net Net-(U2A--): track 41.1 -> 25.8 mm
- net PIN 34: track 48.0 -> 33.1 mm
- net GND: track 139.2 -> 129.5 mm
- net Net-(U2A-+): track 51.2 -> 54.3 mm
- net Net-(R3-Pad2): track 65.6 -> 62.7 mm
